File: rcc-pico/rcc-pico.kicad_sch (KiCad schematic)
At the start: 52 parts, among them J1 Conn_02x02_Odd_Even, J10 Conn_02x04_Odd_Even, J11 Conn_02x04_Odd_Even, J12 Conn_02x04_Odd_Even, J14 Conn_02x05_Odd_Even, J15 Conn_02x02_Odd_Even, J16 Conn_01x02_Pin, J3 PJ-006A, J5 Conn_3x4_female, J7 Conn_03x10, J8 Screw_Terminal, Q1 BSS138, Q2 BSS138, Q3 BSS138, SW1 SW_Push, SW2 SW_Push, U1 AP63300WU-7, U2 AP2115M-3.3TRG1, U3 PicoW

Commit message: finished DRC, added fiducals and name, cleaned up schematic a bit, still needs some work
Parts:
- removed J15: Conn_02x02_Odd_Even, Connector_PinSocket_2.54mm:PinSocket_2x02_P2.54mm_Vertical, symbol Connector_Generic:Conn_02x02_Odd_Even
Connections:
- no-connect marks 20 -> 16
Other:
- note added: "*EXTRAS*"
- note added: "5V Buck Converter"
- note added: "GPIO 0-13"
- note added: "GPIO 14&15 I2C1 Expansion"
- note added: "GPIO 16-18 5V PWM activate"
- note added: "can connect adcref to board's 3v3"
- note added: "require connecting pins to corresponding gpio"
- note added: "~5V PWM OUT"
- note removed: "5V Buck"
- note removed: "5V PWM activate"
- note removed: "I2C1 Activate GPIO 14&15"
- note removed: "Servo Connection (3x3)"
- note removed: "add fadusials for pick and place"
- note removed: "gpio options for I2C1 bus SCL: 3 7 11 15 19 SDA: 2 6 10 14 18"
- note removed: "leaving unconnected so switch must be on to power the devices, not all from pico"
- note removed: "notes: SPI1, I2C0, UART0 used for wifi going to breakout I2C1"
- note removed: "notes: flip switch labels"
- note removed: "options for PWM 0 1 4 5 8 9 12 13 16 17 20 21 22"
- note removed: "this allows for gpio to be used and expansion pins to be used *must activate breakouts to only use one at a time"
- note removed: "use shunt to connect adcref to board's 3v3"
- moved on the sheet: C5, C7, C8, C9, D1, D2, H1, H2, H3, H4, J1, J10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
